File: TESTFREENFET3.sch (EAGLE design)
At the start: 21 parts, among them J1 Digital_0_7, J2 Analog, J3 Digital_8_13

Commit message: Created TESTFREENFET3 project for release v1.0
Parts:
- removed SL1: Digital_0_7, freetronics:M08
- removed SL2: Analog, freetronics:M06SIP
- removed SL3: Digital_8_13, freetronics-original:M100.1
- removed SLP: Power, freetronics:M08
- added C1: 1uF 0603, freetronics-master-v1:CAP0603
- added IC1: WS2811-SOP8, freetronics-jon:WS2811-SOP8
- added JP2: DRAIN3, freetronics-jon:M012.1MM
- added JP3: DRAIN1, freetronics-jon:M012.1MM
- added JP4: SOURCE, freetronics-jon:M012.1MM
- added JP5: IN, freetronics-jon:M03PTH
- added JP6: OUT, freetronics-jon:M03PTH
- added PIEZO2: PIEZOPOLARISED, freetronics-jon:PIEZOPOLARISED
- added R6, R7, R8: 1K, freetronics-jon:RESISTOR0603
- JP1: value MODULE -> DRAIN2; device freetronics-master-v1.1:M04PTH -> freetronics-jon:M012.1MM
- R1, R2, R3: value 560R 0603 -> 560R
- R4: value 1K 0603 -> 1K
- R5: value 1K5 0603 -> 1K5
Connections:
- new net DIN: IC1.DIN, JP6.2
- new net N$5: JP3.1, R6.2
- new net N$6: JP1.1, R7.2
- new net N$8: JP2.1, R8.2
- new net OUT2: IC1.G
- new net OUT3: IC1.B
- net 3V3: no longer SLP.4
- net 5V: no longer SLP.5
- net A0: no longer SL2.1
- net A1: no longer SL2.2
- net A2: no longer SL2.3
- net A3: no longer SL2.4
- net A4: no longer SL2.5
- net A5: no longer SL2.6
- net AREF: no longer SL3.8
- net D0_RX: no longer SL1.1
- net D10: now also R8.1; no longer SL3.3
- net D11_MOSI: now also R7.1; no longer SL3.4
- net D12_MISO: no longer SL3.5
- net D13_SCK: no longer SL3.6
- net D1_TX: no longer SL1.2
- net D2: no longer SL1.3
- net D3: no longer SL1.4
- net D4: no longer SL1.5
- net D5: now also JP5.2; no longer SL1.6
- net D6: now also R6.1; no longer SL1.7
- net D7: now also IC1.R; no longer SL1.8
- net D8: no longer SL3.1
- net D9: now also PIEZO2.+; no longer SL3.2
- net GND: now also C1.2, IC1.GND, JP4.1, JP5.3, JP6.3, PIEZO2.-; no longer JP1.1, SL3.7, SLP.6, SLP.7
- net IOREF: now also C1.1, IC1.SET, IC1.VDD, JP5.1, JP6.1; no longer JP1.4, SLP.2
- net NC: no longer SLP.1
- net RESET: no longer SLP.3
- net SCL: no longer JP1.3, SL3.10
- net SDA: no longer JP1.2, SL3.9
- net VIN: no longer SLP.8
Other:
- note added: "-->"
- note added: "D2: GREEN D3: YELLOW D4: RED D5: TESTDATA D6: TESTSENSE1 D7: OUTPUTSENSE D8: DETECT D9: PIEZO D11: TESTSENSE2 D10: TESTSENSE3"
- note added: "DETECT"
- note added: "Freetronics FREENFET3 Test Shield"
- note added: "GREEN"
- note added: "OUTPUTSENSE"
- note added: "PIEZO"
- note added: "Place module here"
- note added: "Pull-up in software"
- note added: "RED"
- note added: "SKU: TESTFREENFET3"
- note added: "TESTDATA"
- note added: "TESTSENSE"
- note added: "V1.0 (2017-09-13)"
- note added: "YELLOW"
- note added: "tron.cc/freenfet3"
- note removed: "Freetronics I2C Test Shield"
- note removed: "SKU: TESTI2C"
- note removed: "V1.0 (2014-06-24)"
- note removed: "tron.cc/testi2c"
- moved on the sheet: J1, J2, J3, LED1, LED2, LED3, LED4, PIEZO, POWER, R1, R2, R3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
